Commit message: NewReadWay

File: URDFs/URDF_description/urdf/URDF.xacro (robot description, xacro)
@@ -559,4 +559,5 @@
   <child link="Front_leg_left_v4_Spiegeln__1"/>
   <axis xyz="-1.0 0.0 -0.0"/>
+  <!-- <axis xyz="1.0 0.0 -0.0"/> -->
   <limit upper="1.047198" lower="-1.570796" effort="100" velocity="100"/>
 </joint>
@@ -566,4 +567,5 @@
   <child link="Upper_Leg_v5_1"/>
   <axis xyz="1.0 0.0 0.0"/>
+  <!-- <axis xyz="-1.0 0.0 0.0"/> -->
   <limit upper="0.174533" lower="-2.268928" effort="100" velocity="100"/>
 </joint>
@@ -587,5 +589,7 @@
   <child link="Lower_Leg_v2_1"/>
   <axis xyz="-1.0 -0.0 -0.0"/>
-  <limit upper="1.047198" lower="-0.785398" effort="100" velocity="100"/>
+  <!-- <axis xyz="1.0 -0.0 -0.0"/> -->
+  <!-- <limit upper="1.047198" lower="-0.785398" effort="100" velocity="100"/> -->
+  <limit upper="0.785398" lower="-1.047198" effort="100" velocity="100"/>
 </joint>
 <joint name="Umdrehung 14" type="revolute">
@@ -594,4 +598,5 @@
   <child link="Foot_v4__1__1"/>
   <axis xyz="-1.0 -0.0 -0.0"/>
+  <!-- <axis xyz="1.0 -0.0 -0.0"/> -->
   <limit upper="0.785398" lower="-0.785398" effort="100" velocity="100"/>
 </joint>

Commit message: ImproveRL_Training_v1

File: URDFs/URDF_description/urdf/URDF.xacro (robot description, xacro)
@@ -147,5 +147,5 @@
   <inertial>
     <origin xyz="0.01000405917651935 0.01418921203389055 0.04202307290944826" rpy="0 0 0"/>
-    <mass value="0.08505795784466541"/>
+    <mass value="0.02505795784466541"/>
     <inertia ixx="0.00019" iyy="9.4e-05" izz="0.000141" ixy="-0.0" iyz="6.4e-05" ixz="0.0"/>
   </inertial>
@@ -327,5 +327,5 @@
   <inertial>
     <origin xyz="8.382534673334607e-08 0.010542383576317621 0.0026915588221251823" rpy="0 0 0"/>
-    <mass value="0.011213792729013291"/>
+    <mass value="0.101"/>
     <inertia ixx="1e-06" iyy="1e-06" izz="1e-06" ixy="-0.0" iyz="0.0" ixz="0.0"/>
   </inertial>
